File: Plate/Z18_Plate.kicad_pcb (KiCad board)
At the start: 2 copper layers, 371.5 x 100 mm, 17 parts, among them J4 C165948_-_USB_C_Receptacle_US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, SW14 BCKSP, SW36 np_plus, SW52 ENT, SW72 np_ent, SW76 SPC_6.25U

Commit message: JLC rev1 order placed
Parts:
- removed BATT1: SW_SPDT, COBoards_parts:SW-TH_MSK12C02_access_cutout
- removed D50: D, Diode_SMD:D_SOD-123
- removed D83, D86: LED, COBoards_parts:LED_0603_1608Metric_Window
- removed H10, H13, H3, H5, H7: MountingHole_Pad, MountingHole:MountingHole_2.2mm_M2
- removed J4: C165948_-_USB_C_Receptacle_USB2.0_SMD, Connector_USB:USB_C_Receptacle_HRO_TYPE-C-31-M-12
- removed REF**: MX_2.25U, COBoards_parts:MX_2.25U
- removed RESET1: SW_Push, Button_Switch_SMD:SW_SPST_B3U-1000P
- removed SW14: BCKSP, COBoards_parts:MX_2U
- removed SW36: np_plus, COBoards_parts:MX_1U_plate_cutout
- removed SW52: ENT, COBoards:MX_2.25U
- removed SW72: np_ent, COBoards_parts:MX_1U_plate_cutout
- removed SW76: SPC_6.25U, COBoards:MX_6.25U
Routing:
- net Net-(C5-Pad2): track 16.4 -> 0.00 mm
- net /VBUS: track 13.6 -> 0.00 mm
- net GND: track 7.41 -> 0.00 mm, vias 78 -> 0
- net Net-(J4-PadA7): track 3.14 -> 0.00 mm
- net Net-(J4-PadA6): track 3.09 -> 0.00 mm
- removed copper zone on B.Cu, net GND
- removed copper zone on F.Cu, net GND
Other:
- board size 371.5 x 100 mm -> 385.8 x 116.7 mm
- board text removed: "+"
- board text removed: "-"
- board text removed: "->"
- board text removed: "1.5U"
- board text removed: "1U"
- board text removed: "JLCJLCJLC"
- board text removed: "MODEL: Z18 REVISION: 1 DATE: 28 NOV 2021 BY: GITHUB.COM/ERICRLAU"
- board text removed: "OFF ON"
- board text removed: "RESET"
- board text removed: "STANDARD"
- board text removed: "STEPPED"
